File: hardware/XIAO-LiFePO4-Power-Module.kicad_pcb (KiCad board)
At the start: 2 copper layers, 18.5 x 21 mm, 23 parts, among them IC1 RT6150B-33GQW, IC2 APX810S-31SA-7, J1 Conn_JST-XH_1x2, J2 Conn_Castellation_1x3, J7 Conn_Castellation_1x2_no_GND, Q1 AO3415, SW1 Switch, U1 TP5000-QFN16

Commit message: Save
Other:
- board text added: "XIAO-LiFePO4 Power-Module V1.0"
- board text removed: "LiFePO4 charge-discharge Module V1.0"
Changed lines of the file:
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@@
 		)
 	)
-	(gr_text "LiFePO4\ncharge-discharge\nModule V1.0"
-		(at 36.07 26.96 0)
+	(gr_text "XIAO-LiFePO4\nPower-Module\nV1.0"
+		(at 36.1 29.3 0)
 		(layer "B.SilkS")
 		(effects
